File: pcb9segCounter/9SegDigit.kicad_sch (KiCad schematic)
At the start: 19 parts

Commit message: Doing lots of cleanup
Other:
- note added: "9-Segment Window"
- note added: "Segment Decoupling Capacitors"
- note added: "Segment Neopixels: SK6805 EC10"
- note removed: "SK6805 EC10"
- company: (none) -> Ryan Martin
- title: (none) -> Nine Segment SAO
- moved on the sheet: C10, C11, C12, C13, C14, C15, C16, C17, C18, D10, D11, D12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
